Commit message: Fix safety findings from the adversarial review
Firmware:
- JOINT_STREAM bypasses the VR low-pass filter: with alpha < 1 (wrist
  pitch/roll = 0.35 at boot) the output followed the EMA of the target and
  ignored the rate limit, so wrist jumps were possible
- JOINT_STREAM speed is a fixed 60 deg/s (per-joint caps still apply), no
  longer inherited from the VR speed buttons / SET_VR_PARAMS
- JOINT_STREAM never re-arms SAFE -> IDLE automatically: after UART SAFE,
  E-STOP recovery or an SPI watchdog trip the still-running stream would
  have driven the arm back to its last target; an explicit ENABLE is needed
- the stream servo-disable latch is reset when leaving mode 6

Pi / ROS 2:
- Jonny5System: STREAM_ENABLE consent gate (IDLE, no E-STOP, command within
  arm_gate_rad of the pose when (re)arming); consent withdrawn whenever the
  firmware leaves IDLE
- spi_driver_node: joint_stream/enable refuses stale (>0.5 s) or far
  (>0.05 rad) commands and a non-IDLE/E-STOP firmware; streaming is
  disabled automatically when the firmware leaves IDLE
- URDF/ros2_control limits aligned with the firmware clamps (wrist pitch
  -45..30 deg, wrist roll -45..40 deg)
- intent_to_servo publishes one zero twist on deadman release
- mock SPI keeps joints still when not streaming; sim_e2e covers the
  refusal/acceptance of joint_stream/enable and is more robust to timing
- docs and hardware test plan updated (explicit UART ENABLE, new checks)

Co-Authored-By: Claude Opus 5.5 <noreply@anthropic.com>
Claude-Session: https://claude.ai/code/session_0147uyWzMg28ez6ehh9LPKvA

File: ros2_ws/src/jonny5_description/urdf/jonny5.ros2_control.xacro (robot description, xacro)
@@ -35,6 +35,6 @@
       <xacro:jonny5_joint_interfaces name="elbow_joint" lower="-1.047198" upper="0.959931" />
       <xacro:jonny5_joint_interfaces name="wrist_yaw_joint" lower="-0.785398" upper="0.785398" />
-      <xacro:jonny5_joint_interfaces name="wrist_pitch_joint" lower="-0.959931" upper="0.523599" />
-      <xacro:jonny5_joint_interfaces name="wrist_roll_joint" lower="-0.785398" upper="0.785398" />
+      <xacro:jonny5_joint_interfaces name="wrist_pitch_joint" lower="-0.785398" upper="0.523599" />
+      <xacro:jonny5_joint_interfaces name="wrist_roll_joint" lower="-0.785398" upper="0.698132" />
       <sensor name="imu_sensor">
         <state_interface name="orientation.x" />

File: ros2_ws/src/jonny5_description/urdf/jonny5.urdf.xacro (robot description, xacro)
@@ -74,5 +74,6 @@
     <origin xyz="0 0 ${wrist_stack/3}" rpy="0 0 0" />
     <axis xyz="0 1 0" />
-    <limit lower="-0.959931" upper="0.523599" effort="2.0" velocity="1.5" />
+    <!-- Firmware clamps pitch to 45..135 deg physical (offset 90, dir -1) -> -45..+45 deg. -->
+    <limit lower="-0.785398" upper="0.523599" effort="2.0" velocity="1.5" />
   </joint>
   <link name="wrist_roll_link"><visual><origin xyz="0 0 ${wrist_stack/3}" /><geometry><box size="0.030 0.030 ${wrist_stack/3}" /></geometry><material name="jonny5_dark" /></visual></link>
@@ -82,5 +83,6 @@
     <origin xyz="0 0 ${wrist_stack/3}" rpy="0 0 0" />
     <axis xyz="1 0 0" />
-    <limit lower="-0.785398" upper="0.785398" effort="2.0" velocity="1.5" />
+    <!-- Firmware clamps roll to 45..135 deg physical (offset 95) -> -50..+40 deg. -->
+    <limit lower="-0.785398" upper="0.698132" effort="2.0" velocity="1.5" />
   </joint>
   <link name="ee_link"><visual><origin xyz="${tool_x/2} 0 0" /><geometry><box size="${tool_x} 0.025 0.025" /></geometry><material name="jonny5_signal" /></visual></link>
