Commit message: URDF: wrist geometry from the POE model used by the legacy FK/IK
The URDF did not match the robot. The pitch axis was 57 mm too high (the
roll joint sat 57 mm above it) and the tool point 115 mm above the pitch
axis instead of 57 mm in front of it: tool position errors up to 171 mm.
Cartesian commands (MoveIt Servo) were computed for the wrong point.

New geometry, from the POE parameters on the settings page (shoulder axis
134.3 mm, elbow 194.3 mm, wrist pitch 381.225 mm, roll axis along x through
the pitch point, tool 57 mm forward): URDF forward kinematics world ->
ee_link now matches the POE product of exponentials with 0.0000 mm error
over 1000 random poses. Only the wrist links, the forearm length and the
shoulder height (112.3 mm + 22 mm plinth) change; axes, limits and joint
names are unchanged, so offsets, signs and the SRDF poses still apply.

Note: j5_poe_params.json on the Pi still holds older values (112/172/345
mm); the settings page save did not reach it while ws-teleop was stopped.

Co-Authored-By: Claude Opus 5.5 <noreply@anthropic.com>

File: ros2_ws/src/jonny5_description/urdf/jonny5.urdf.xacro (robot description, xacro)
@@ -6,8 +6,15 @@
   <xacro:arg name="spi_device" default="/dev/spidev0.0" />
   <xacro:arg name="transfer_len" default="128" />
-  <xacro:property name="base_height" value="0.112" />
+  <!-- Geometry from the POE model used by the legacy FK/IK
+       (raspberry/config_runtime/kinematics/j5_poe_params.json, settings page):
+       shoulder axis at 134.3 mm (22 mm plinth + base_height), elbow 60 mm above it,
+       wrist pitch axis at 381.225 mm, roll axis along x through the pitch point,
+       tool point 57 mm forward of it (M). The yaw axis is vertical through x=0; its
+       height does not change the kinematics (yaw_to_pitch is only for the visual). -->
+  <xacro:property name="base_height" value="0.1123" />
   <xacro:property name="upper_arm" value="0.060" />
-  <xacro:property name="forearm" value="0.173" />
-  <xacro:property name="wrist_stack" value="0.172" />
+  <xacro:property name="elbow_to_pitch" value="0.186925" />
+  <xacro:property name="yaw_to_pitch" value="0.057" />
+  <xacro:property name="forearm" value="${elbow_to_pitch - yaw_to_pitch}" />
   <xacro:property name="tool_x" value="0.057" />
   <material name="jonny5_dark"><color rgba="0.08 0.09 0.10 1.0" /></material>
@@ -60,5 +67,5 @@
     <limit lower="-1.047198" upper="0.959931" effort="5.0" velocity="1.5" />
   </joint>
-  <link name="wrist_yaw_link"><visual><origin xyz="0 0 ${wrist_stack/3}" /><geometry><box size="0.035 0.035 ${wrist_stack/3}" /></geometry><material name="jonny5_dark" /></visual></link>
+  <link name="wrist_yaw_link"><visual><origin xyz="0 0 ${yaw_to_pitch/2}" /><geometry><box size="0.035 0.035 ${yaw_to_pitch}" /></geometry><material name="jonny5_dark" /></visual></link>
   <joint name="wrist_yaw_joint" type="revolute">
     <parent link="forearm_link" />
@@ -68,27 +75,28 @@
     <limit lower="-0.785398" upper="0.785398" effort="2.0" velocity="1.5" />
   </joint>
-  <link name="wrist_pitch_link"><visual><origin xyz="0 0 ${wrist_stack/3}" /><geometry><box size="0.032 0.032 ${wrist_stack/3}" /></geometry><material name="jonny5_signal" /></visual></link>
+  <link name="wrist_pitch_link"><visual><geometry><box size="0.032 0.040 0.032" /></geometry><material name="jonny5_signal" /></visual></link>
   <joint name="wrist_pitch_joint" type="revolute">
     <parent link="wrist_yaw_link" />
     <child link="wrist_pitch_link" />
-    <origin xyz="0 0 ${wrist_stack/3}" rpy="0 0 0" />
+    <origin xyz="0 0 ${yaw_to_pitch}" rpy="0 0 0" />
     <axis xyz="0 1 0" />
     <!-- Firmware clamps pitch to 45..135 deg physical (offset 90, dir -1) -> -45..+45 deg. -->
     <limit lower="-0.785398" upper="0.523599" effort="2.0" velocity="1.5" />
   </joint>
-  <link name="wrist_roll_link"><visual><origin xyz="0 0 ${wrist_stack/3}" /><geometry><box size="0.030 0.030 ${wrist_stack/3}" /></geometry><material name="jonny5_dark" /></visual></link>
+  <link name="wrist_roll_link"><visual><origin xyz="${tool_x/2} 0 0" /><geometry><box size="${tool_x} 0.025 0.025" /></geometry><material name="jonny5_dark" /></visual></link>
   <joint name="wrist_roll_joint" type="revolute">
     <parent link="wrist_pitch_link" />
     <child link="wrist_roll_link" />
-    <origin xyz="0 0 ${wrist_stack/3}" rpy="0 0 0" />
+    <!-- Roll axis (x) passes through the pitch point: no offset. -->
+    <origin xyz="0 0 0" rpy="0 0 0" />
     <axis xyz="1 0 0" />
     <!-- Firmware clamps roll to 45..135 deg physical (offset 95) -> -50..+40 deg. -->
     <limit lower="-0.785398" upper="0.698132" effort="2.0" velocity="1.5" />
   </joint>
-  <link name="ee_link"><visual><origin xyz="${tool_x/2} 0 0" /><geometry><box size="${tool_x} 0.025 0.025" /></geometry><material name="jonny5_signal" /></visual></link>
+  <link name="ee_link"><visual><geometry><sphere radius="0.008" /></geometry><material name="jonny5_signal" /></visual></link>
   <joint name="tool_joint" type="fixed">
     <parent link="wrist_roll_link" />
     <child link="ee_link" />
-    <origin xyz="0 0 ${wrist_stack/3}" rpy="0 0 0" />
+    <origin xyz="${tool_x} 0 0" rpy="0 0 0" />
   </joint>
   <link name="imu_link" />

Commit message: Align URDF limits, elbow dir and poses with the dashboard settings
Checked the dashboard settings against the hardware test:

- URDF joint limits: intersection of the previous limits and the
  dashboard limits that ws-teleop loads into the firmware at boot
  (routing_config.json, physical deg). The firmware clamps outside them,
  so ROS could command angles the arm never reached (base up to +45 deg
  vs +35, wrist pitch -45 deg vs -30 ...). Base +35, shoulder -57,
  elbow +52, wrist yaw +40, wrist pitch -30..+30 deg.
- config_runtime/robot/j5_settings.json: elbow dir -1 -> +1 (phase 4:
  servo + moves the forearm forward, positive about +y in the POE/URDF).
  The elbow angle of every stored pose was converted (virtual -> 180 -
  virtual) so the physical poses are unchanged. Demo steps 5 and 6 were
  outside the dashboard limits (base 146, elbow 15 physical) and are now
  at the limits (135, 30).
- config_runtime/kinematics/j5_poe_params.json: the POE saved from the
  settings page (shoulder 134.3, elbow 194.3, wrist 381.225 mm, tool 57 mm).

Both config files are copies of the live files on the Pi. sim_e2e ALL PASS.

Co-Authored-By: Claude Opus 5.5 <noreply@anthropic.com>

File: ros2_ws/src/jonny5_description/urdf/jonny5.urdf.xacro (robot description, xacro)
@@ -41,5 +41,10 @@
     <origin xyz="0 0 0.022" rpy="0 0 0" />
     <axis xyz="0 0 1" />
-    <limit lower="-0.785398" upper="0.785398" effort="5.0" velocity="2.0" />
+    <!-- Joint limits: intersection of the previous URDF limits and the dashboard
+         limits that ws-teleop loads into the firmware at boot (routing_config.json,
+         physical deg, converted with offsets 100 88 93 95 90 95 and dirs 1 -1 1 1 -1 1).
+         The firmware clamps outside them, so ROS must not command beyond.
+         Base: dashboard 45..135 phys -> -55..+35 deg. -->
+    <limit lower="-0.785398" upper="0.610865" effort="5.0" velocity="2.0" />
   </joint>
   <link name="upper_arm_link">
@@ -53,5 +58,6 @@
     <origin xyz="0 0 ${base_height}" rpy="0 0 0" />
     <axis xyz="0 1 0" />
-    <limit lower="-1.047198" upper="0.959931" effort="5.0" velocity="1.5" />
+    <!-- Dashboard 30..145 phys -> -57..+58 deg. -->
+    <limit lower="-0.994838" upper="0.959931" effort="5.0" velocity="1.5" />
   </joint>
   <link name="forearm_link">
@@ -65,5 +71,6 @@
     <origin xyz="0 0 ${upper_arm}" rpy="0 0 0" />
     <axis xyz="0 1 0" />
-    <limit lower="-1.047198" upper="0.959931" effort="5.0" velocity="1.5" />
+    <!-- Dashboard 30..145 phys -> -63..+52 deg. -->
+    <limit lower="-1.047198" upper="0.907571" effort="5.0" velocity="1.5" />
   </joint>
   <link name="wrist_yaw_link"><visual><origin xyz="0 0 ${yaw_to_pitch/2}" /><geometry><box size="0.035 0.035 ${yaw_to_pitch}" /></geometry><material name="jonny5_dark" /></visual></link>
@@ -73,5 +80,6 @@
     <origin xyz="0 0 ${forearm}" rpy="0 0 0" />
     <axis xyz="0 0 1" />
-    <limit lower="-0.785398" upper="0.785398" effort="2.0" velocity="1.5" />
+    <!-- Dashboard 45..135 phys -> -50..+40 deg. -->
+    <limit lower="-0.785398" upper="0.698132" effort="2.0" velocity="1.5" />
   </joint>
   <link name="wrist_pitch_link"><visual><geometry><box size="0.032 0.040 0.032" /></geometry><material name="jonny5_signal" /></visual></link>
@@ -81,6 +89,7 @@
     <origin xyz="0 0 ${yaw_to_pitch}" rpy="0 0 0" />
     <axis xyz="0 1 0" />
-    <!-- Firmware clamps pitch to 45..135 deg physical (offset 90, dir -1) -> -45..+45 deg. -->
-    <limit lower="-0.785398" upper="0.523599" effort="2.0" velocity="1.5" />
+    <!-- Dashboard 35..120 phys (offset 90, dir -1) -> -30..+55 deg; firmware default
+         45..135 -> -45..+45. Intersection with the previous URDF range: -30..+30. -->
+    <limit lower="-0.523599" upper="0.523599" effort="2.0" velocity="1.5" />
   </joint>
   <link name="wrist_roll_link"><visual><origin xyz="${tool_x/2} 0 0" /><geometry><box size="${tool_x} 0.025 0.025" /></geometry><material name="jonny5_dark" /></visual></link>
@@ -91,5 +100,5 @@
     <origin xyz="0 0 0" rpy="0 0 0" />
     <axis xyz="1 0 0" />
-    <!-- Firmware clamps roll to 45..135 deg physical (offset 95) -> -50..+40 deg. -->
+    <!-- Dashboard and firmware 45..135 phys (offset 95) -> -50..+40 deg. -->
     <limit lower="-0.785398" upper="0.698132" effort="2.0" velocity="1.5" />
   </joint>

Commit message: URDF: wrist pitch upper limit +45 deg so PARK (+40 deg) is inside
The intersection in the previous commit capped pitch at +30 deg, but the
dashboard allows up to +55 deg (35 phys) and PARK uses +40 deg: MoveIt
would treat PARK as out of bounds. +45 deg is inside the dashboard limit
and the firmware default range. PARK checked on the robot and in RViz.

Co-Authored-By: Claude Opus 5.5 <noreply@anthropic.com>

File: ros2_ws/src/jonny5_description/urdf/jonny5.urdf.xacro (robot description, xacro)
@@ -90,6 +90,6 @@
     <axis xyz="0 1 0" />
     <!-- Dashboard 35..120 phys (offset 90, dir -1) -> -30..+55 deg; firmware default
-         45..135 -> -45..+45. Intersection with the previous URDF range: -30..+30. -->
-    <limit lower="-0.523599" upper="0.523599" effort="2.0" velocity="1.5" />
+         45..135 -> -45..+45. Intersection: -30..+45 (PARK uses +40, tip down). -->
+    <limit lower="-0.523599" upper="0.785398" effort="2.0" velocity="1.5" />
   </joint>
   <link name="wrist_roll_link"><visual><origin xyz="${tool_x/2} 0 0" /><geometry><box size="${tool_x} 0.025 0.025" /></geometry><material name="jonny5_dark" /></visual></link>
